File: quadrature/quadrature.kicad_pcb (KiCad board)
At the start: 2 copper layers, 100 x 100 mm, 6 parts, among them J1 Screw_Terminal_01x05, J2 Conn_02x20_Counter_Clockwise, U1 4013, U2 4029, U3 4029, U4 4029

Commit message: Improve routing
Connections:
- J1 pad 2: /ENC_B -> Vss
- J1 pad 3: /ENC_A -> Vss
- U1 pad 3: /ENC_A -> Vss
- U1 pad 5: /ENC_B -> Vss
- U2 pad 15: /ENC_A -> Vss
- U3 pad 15: /ENC_A -> Vss
- U4 pad 15: /ENC_A -> Vss
Routing:
- net Vss: track 221.0 -> 368.7 mm
- net /ENC_A: track 134.9 -> 0.00 mm, vias 1 -> 0
- net /ENC_B: track 15.2 -> 0.00 mm
- net Net-(U1-Pad1): track 179.8 -> 172.1 mm, vias 6 -> 5
- net Net-(U2-Pad7): track 41.8 -> 34.5 mm
- net Net-(J2-Pad18): track 48.3 -> 44.2 mm, vias 1 -> 0
- net Net-(J2-Pad8): track 42.4 -> 43.2 mm, vias 2 -> 1
- net Net-(J2-Pad12): track 42.8 -> 42.1 mm, vias 1 -> 0
- net Net-(J2-Pad14): vias 3 -> 1
