File: quadrature/quadrature.kicad_sch (KiCad schematic)
At the start: 6 parts, among them U1 4013, U3 4029, U4 4029

Commit message: Improve routing
Parts:
- J1: value (none) -> Screw_Terminal_01x05; footprint (none) -> TerminalBlock:TerminalBlock_bornier-5_P5.08mm
- J2: value (none) -> Conn_02x20_Counter_Clockwise; footprint (none) -> Connector_IDC:IDC-Header_2x20_P2.54mm_Vertical
- U1: footprint (none) -> Package_DIP:DIP-14_W7.62mm_LongPads
- U2: value (none) -> 4029; footprint (none) -> Package_DIP:DIP-16_W7.62mm_LongPads
- U3, U4: footprint (none) -> Package_DIP:DIP-16_W7.62mm_LongPads
Connections:
- net ENC_A is gone; now on net Vss: J1.3 (Pin_3), U1.3 (Cp), U2.15 (CK), U3.15 (CK), U4.15 (CK)
- net ENC_B is gone; now on net Vss: J1.2 (Pin_2), U1.5 (D)
Other:
- moved on the sheet: J1, J2, U1A, U1B, U2, U3, U4
